File: motor_driver_board/KORSAK-8-wheel.sch (KiCad schematic (older format))
At the start: 16 parts, among them J1 Screw_Terminal_01x04, J2 Conn_01x02_Male, J3 Screw_Terminal_01x06, J4 Screw_Terminal_01x04, M1 Motor_DC, M2 Motor_DC, M3 Motor_DC, M4 Motor_DC, M5 Motor_DC, M6 Motor_DC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

Commit message: Переместил файлы
Parts:
- removed J1, J4: Screw_Terminal_01x04, TerminalBlock_Phoenix:TerminalBlock_Phoenix_MKDS-1,5-4_1x04_P5.00mm_Horizontal, symbol Connector:Screw_Terminal_01x04
- added J1: Screw_Terminal_01x06, TerminalBlock_Phoenix:TerminalBlock_Phoenix_MKDS-1,5-6_1x06_P5.00mm_Horizontal, symbol Connector:Screw_Terminal_01x06
Connections:
- net labels added: +BATT
- wire segments 149 -> 123

Commit message: Синхронизировал историю коммитов с master веткой
Parts:
- added C1, C2, C3, C4, C5, C6, C7, C8: 10pF, Capacitor_THT:C_Disc_D5.0mm_W2.5mm_P5.00mm, symbol Device:C
Connections:
- net at M4.1 (+), U4.11 (3Y): now also C6.1
- net at M4.2 (-), U4.14 (4Y): now also C6.2
- net at M3.1 (+), U4.3 (1Y): now also C5.1
- net at M3.2 (-), U4.6 (2Y): now also C5.2
- net at M2.1 (+), U1.11 (3Y): now also C2.1
- net at M2.2 (-), U1.14 (4Y): now also C2.2
- net at M1.1 (+), U1.3 (1Y): now also C1.1
- net at M1.2 (-), U1.6 (2Y): now also C1.2
- net at M8.1 (+): now also U2.6 (2Y), C8.1; no longer U2.3 (1Y)
- net at M8.2 (-): now also U2.3 (1Y), C8.2; no longer U2.6 (2Y)
- net at M7.1 (+): now also U2.14 (4Y), C7.1; no longer U2.11 (3Y)
- net at M7.2 (-): now also U2.11 (3Y), C7.2; no longer U2.14 (4Y)
- net at U3.11 (3Y): now also M5.2 (-), C3.2; no longer M5.1 (+)
- net at U3.14 (4Y): now also M5.1 (+), C3.1; no longer M5.2 (-)
- net at U3.3 (1Y): now also M6.2 (-), C4.2; no longer M6.1 (+)
- net at U3.6 (2Y): now also M6.1 (+), C4.1; no longer M6.2 (-)
Other:
- moved on the sheet: J1, J2, J3, M1, M2, M3, M4, M5, M6, M7, M8, U1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
